Commit message: update azure urdf

File: husky_panda_description/urdf/azure_kinect.urdf.xacro (robot description, xacro)
@@ -1,32 +1,53 @@
 <?xml version="1.0"?>
-<robot name="azure-kinect" xmlns:xacro="http://www.ros.org/wiki/xacro">
-  <link name="camera_base">
-    <visual>
-      <origin rpy="1.5708 0 1.5708" xyz="-0.0259 0 0"/>
-      <geometry>
-        <mesh filename="package://husky_panda_description/meshes/Azure_Kinect_DK.stl" scale="0.001 0.001 0.001"/>
-      </geometry>
-      <material name="grey">
-        <color rgba="0.6 0.6 0.6 1" />
-      </material>
-    </visual>
-  </link>
-  <link name="depth_camera_link"/>
-  <joint name="cam2base_joint" type="fixed">
-    <parent link="camera_base"/>
-    <child link="depth_camera_link"/>
-    <origin rpy="-1.6755133 0.0000028 -1.5707995" xyz="0 0 0.0018"/>
-  </joint>
-  <link name="imu_camera_link"/>
-  <joint name="depth2imu_joint" type="fixed">
-    <parent link="depth_camera_link"/>
-    <child link="imu_camera_link"/>
-    <origin rpy="-0.0014611 1.4592022 1.5710739" xyz="0.00346563 0.00415245 -0.0507355"/>
-  </joint>
-  <link name="rgb_camera_link"/>
-  <joint name="depth2rgb_joint" type="fixed">
-    <parent link="depth_camera_link"/>
-    <child link="rgb_camera_link"/>
-    <origin rpy="0.1027897 0.0048339 0.0004876" xyz="0.0320149 0.00252428 -0.00366382"/>
-  </joint>
+<robot name="azure_kinect" xmlns:xacro="http://www.ros.org/wiki/xacro">
+  <xacro:macro name="azure_kinect" params="is_reverse:=false">
+    <link name="camera_base">
+      <visual>
+        <origin rpy="1.5708 0 1.5708" xyz="-0.0259 0 0"/>
+        <geometry>
+          <mesh filename="package://husky_panda_description/meshes/Azure_Kinect_DK.stl" scale="0.001 0.001 0.001"/>
+        </geometry>
+        <material name="grey">
+          <color rgba="0.6 0.6 0.6 1" />
+        </material>
+      </visual>
+    </link>
+    <link name="depth_camera_link"/>
+    <link name="imu_camera_link"/>
+    <link name="rgb_camera_link"/>
+    <xacro:unless value="${is_reverse}">
+      <joint name="cam2depth_joint" type="fixed">
+        <parent link="camera_base"/>
+        <child link="depth_camera_link"/>
+        <origin rpy="-1.6755133 0.0000028 -1.5707995" xyz="0 0 0.0018"/>
+      </joint>
+      <joint name="depth2imu_joint" type="fixed">
+        <parent link="depth_camera_link"/>
+        <child link="imu_camera_link"/>
+        <origin rpy="-0.0014611 1.4592022 1.5710739" xyz="0.00346563 0.00415245 -0.0507355"/>
+      </joint>
+      <joint name="depth2rgb_joint" type="fixed">
+        <parent link="depth_camera_link"/>
+        <child link="rgb_camera_link"/>
+        <origin rpy="0.1027897 0.0048339 0.0004876" xyz="0.0320149 0.00252428 -0.00366382"/>
+      </joint>
+    </xacro:unless>
+    <xacro:if value="${is_reverse}">
+      <joint name="rgb2depth_joint" type="fixed">
+        <parent link="rgb_camera_link"/>
+        <child link="depth_camera_link"/>
+        <origin rpy="-0.102789 -0.004858 0.000011" xyz="-0.032033 -0.002135 0.003748"/>
+      </joint>
+      <joint name="depth2imu_joint" type="fixed">
+        <parent link="depth_camera_link"/>
+        <child link="imu_camera_link"/>
+        <origin rpy="-0.0014611 1.4592022 1.5710739" xyz="0.00346563 0.00415245 -0.0507355"/>
+      </joint>
+      <joint name="depth2cam_joint" type="fixed">
+        <parent link="depth_camera_link"/>
+        <child link="camera_base"/>
+        <origin rpy="-3.141565 -1.466079 -1.570827" xyz="0 0.001790 0.000188"/>
+      </joint>
+    </xacro:if>
+  </xacro:macro>
 </robot>

File: husky_panda_description/urdf/husky_panda.urdf.xacro (robot description, xacro)
@@ -44,5 +44,5 @@
   </xacro:unless>
   <!-- For Azure Kinect -->
-  <link name="kinect_suppot_link">
+  <!-- <link name="kinect_suppot_link">
     <visual>
       <origin rpy="0 0 0" xyz="0 0 0"/>
@@ -59,13 +59,14 @@
     <child link="kinect_suppot_link"/>
     <origin rpy="2.1817 0 1.5708" xyz="-0.0892 0.0 1.3723"/>
-  </joint>
+  </joint> -->
   <xacro:include filename="$(find husky_panda_description)/urdf/azure_kinect.urdf.xacro" />
-  <joint name="kinect_joint" type="fixed">
+  <xacro:azure_kinect is_reverse="true" />
+  <!-- <joint name="kinect_joint" type="fixed">
     <parent link="kinect_suppot_link"/>
     <child link="camera_base"/>
     <origin rpy="0 -1.5707963 -1.5707963" xyz="0 0 0.0259"/>
-  </joint>
+  </joint> -->
   <xacro:include filename="$(find franka_description)/robots/common/franka_arm.xacro"/>
-  <xacro:franka_arm arm_id="$(arg arm_id)" connected_to="base_link"  xyz="0.3 0.0 0.256" gazebo="false" safety_distance="0.02"
+  <xacro:franka_arm arm_id="$(arg arm_id)" connected_to="base_link"  xyz="0.36 0.0 0.256" gazebo="false" safety_distance="0.02"
   joint_limits="${xacro.load_yaml('$(find franka_description)/robots/panda/joint_limits.yaml')}"/>
   <xacro:if value="$(arg hand)">
@@ -79,3 +80,13 @@
        />
   </xacro:if>
+  <!--rgb camera link to panda_link0
+   [[-0.04882053 -0.63533808  0.77068936 -0.51619329]
+    [-0.99871549  0.04152894 -0.02902973 -0.05741105]
+    [-0.01356222 -0.77111664 -0.63654944  1.10626562]
+    [ 0.          0.          0.          1.        ]] -->
+  <joint name="kinect_joint" type="fixed">
+    <parent link="$(arg arm_id)_link0"/>
+    <child link="rgb_camera_link"/>
+    <origin rpy="-2.2608881 0.0135627 -1.6196408" xyz="-0.51619329 -0.05741105 1.10626562"/>
+  </joint>
 </robot>
